Commit message: dynamical robot

File: contextual_maniskill/assets/robots/panda/panda_v2.urdf (robot description, URDF)
Before this commit: robot panda, 15 links, 14 joints
Joints:
- joint panda_joint5: origin xyz=-1.1825 0.384 0 rpy=-1.5707963267948966 0 0 -> xyz=-0.0825 0.384 0 rpy=-1.5707963267948966 0 0
